File: pcb/mds.brd (EAGLE design)
At the start: 100 x 80 mm, 27 parts, among them U2 ISD1900ISD1932, U3 MICELECTRET_SMD, U4 AUDIO-JACK2SMD

Commit message: Electronique
Parts:
- removed JP4, JP5, JP8: (no value), SparkFun:1X02
- removed JP7: (no value), SparkFun:1X08
- removed JP9: (no value), SparkFun:1X06
- removed S1: (no value), SparkFun:AYZ0202
- removed U$10: ARDUINOMICRO, adafruit:ARDUINOMICRO
- added U$15: ARDUINO_MINI, SparkFun-Boards:ARDUINO_MINI
- moved U$14 134.0 mm to (25.4, 44.5)
- moved U$13 98.8 mm to (44.5, 7.62), turned to 90 degrees
- moved U2 42.4 mm to (36.8, 26.7)
Connections:
- removed net E0: JP7.8, U2.7
- removed net E1: JP7.7, U2.9
- removed net E2: JP7.6, U2.10
- removed net E3: JP7.5, U2.11
- removed net FMC1: JP9.6, U2.6
- removed net FMC2: JP9.5, U2.23
- removed net MODE: S1.2, U2.27
- removed net REC: JP9.4, U2.24
- removed net S0: JP7.4, U2.2
- removed net S1: JP7.3, U2.3
- removed net S2: JP7.2, U2.4
- removed net S3: JP7.1, U2.5
- net 5V: no longer JP4.2, S1.3
- net AGC: no longer JP9.2
- net FT: no longer JP9.1
- net GND: now also U2.27; no longer JP4.1, S1.1
- net LED: no longer JP8.1
- net ROSC: no longer JP9.3
- net SP+: no longer JP5.1
- net SP-: no longer JP5.2
- net XCLK: no longer JP8.2
Routing:
- added copper zone on layer 1, net N$4
Other:
- board size 100 x 80 mm -> 50.5 x 49.5 mm

Commit message: Schema development
Parts:
- removed LED1: Red, SparkFun:LED-0603
- removed U$15: ARDUINO_MINI, SparkFun-Boards:ARDUINO_MINI
- added C12, C14, C15: 0.1uF, SparkFun:0402-CAP
- added JP1: FTDI Basic, SparkFun:1X06
- added JP8: FIDUCIALUFIDUCIAL, SparkFun:MICRO-FIDUCIAL
- added PAD1, PAD2: (no value), wirepad:2,15/1,0
- added Q1: 8/16/20MHz, SparkFun:RESONATOR-SMD
- added R5, R7: (no value), rcl:M0805
- added R6: 10K, SparkFun:0402-RES
- added S2: Reset, SparkFun:TACTILE_SWITCH_SMD
- added T1: (no value), transistor:SOT23-EBC
- added U5: ATMEGA328, SparkFun:TQFP32-08
- R1: value 1k -> (none); device SparkFun:0603-RES -> rcl:M0805
- moved R1 82.8 mm to (2.54, -118.1)
Connections:
- removed net 5V: C1.1, C2.1, C3.1, C4.A, C5.A, C6.A, LED1.A, R2.2, U2.14, U2.21, U2.28
- removed net N$1: LED1.C, R1.2
- removed net XCLK: U2.25
- new net AREF: C14.2, U5.20
- new net DTR: C15.2, JP1.1
- new net M1: U2.2, U5.25
- new net M2: U2.3, U5.26
- new net M3: U2.4, U5.19
- new net M4: U2.5, U5.22
- new net M5: U2.7, U5.2
- new net M6: U2.9, U5.9
- new net M7: U2.10, U5.10
- new net M8: U2.11, U5.11
- new net N$10: Q1.3, U5.7
- new net N$5: R5.2, T1.B
- new net N$7: PAD1.1, T1.C
- new net N$9: Q1.1, U5.8
- new net REC/PLAY: U2.24, U5.12
- new net RESET: C15.1, R6.1, S2.3, S2.4, U5.29
- new net RXI: JP1.3, U5.30
- new net SCL: R7.1, U$13.SCL, U5.28
- new net SDA: R1.1, U$13.SDA, U5.27
- new net TXO: JP1.2, U5.31
- new net VIBRATOR: R5.1
- net GND: now also C12.1, C14.1, JP1.5, JP1.6, Q1.2, S2.1, S2.2, T1.E, U5.21, U5.3, U5.5
- net LED: now also U5.32; no longer R1.1
- net VCC: now also C1.1, C12.2, C2.1, C3.1, C4.A, C5.A, C6.A, JP1.4, PAD2.1, R1.2, R2.2, R6.2, R7.2, U2.14, U2.21, U2.23, U2.25, U2.28, U2.6, U5.18, U5.4, U5.6

Commit message: Schema + PCB
Parts:
- removed C10: 4.7uF, SparkFun:0603-CAP
- removed JP8: FIDUCIALUFIDUCIAL, SparkFun:MICRO-FIDUCIAL
- removed PAD1, PAD2: (no value), wirepad:2,15/1,0
- removed Q1: 8/16/20MHz, SparkFun:RESONATOR-SMD
- removed U3: MICELECTRET_SMD, SparkFun:MIC_ELECTRET_SMD
- removed U4: AUDIO-JACK2SMD, SparkFun:AUDIO-JACK-3.5MM-SMD
- added C11, C16, C17, C18, C19, C20: 100nf, rcl:C0805
- added C13: 22pf, rcl:C0805
- added IC1: MAX1555, maxim:SOT23-5L
- added LIPO+, LIPO-, MOT+, MOT-, PWR+, PWR-, SP+, SP-: (no value), wirepad:2,15/1,0
- added M1: ELECTRET_MICROPHON-F6035AP, microphon:F6035AP
- added Q2: (no value), crystal:HC49UP
- added R8: 10k, rcl:M0805
- added RGB: (no value), con-lstb:MA06-1
- added SJ1: (no value), jumper:SJ_2
- C1, C2, C3, C8, C9: value 0.1uF -> 100nf; device SparkFun:0603-CAP -> rcl:C0805
- C12, C15: value 0.1uF -> 100nf; device SparkFun:0402-CAP -> rcl:C0805
- C14: value 0.1uF -> 22pf; device SparkFun:0402-CAP -> rcl:C0805
- C4, C5, C6, C7: value 10uF -> 10uf; device SparkFun:EIA3216 -> rcl:CT3528
- R2, R3, R4: device SparkFun:0603-RES -> rcl:M0805
- R6: value 10K -> (none); device SparkFun:0402-RES -> rcl:M0805
- moved R7 160.8 mm to (54.0, 29.2)
- moved R1 159.0 mm to (54.0, 32.4)
- moved C12 129.2 mm to (10.8, 24.8), turned to 90 degrees
- moved C15 126.0 mm to (11.4, 21.0), turned to 90 degrees
- moved R6 125.0 mm to (37.5, 10.8), turned to 180 degrees
- moved C14 112.7 mm to (15.2, 8.26)
- moved S2 110.5 mm to (3.81, 26.7), turned to 90 degrees
- moved R5 99.8 mm to (39.4, 36.8)
- moved T1 99.1 mm to (40.6, 40.6)
- moved U5 88.5 mm to (11.4, 14.6), turned to 90 degrees
- moved JP1 80.7 mm to (2.54, 8.89), turned to 90 degrees
- moved C9 72.8 mm to (53.3, 26.0)
- moved C3 67.9 mm to (34.9, 24.8)
- moved R4 65.7 mm to (42.5, 12.7), turned to 270 degrees
- moved R2 64.3 mm to (45.7, 3.17), turned to 270 degrees
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Connections:
- removed net ROSC: U2.20
- new net CHG: IC1.3, U5.1
- new net MOSI: RGB.4, U5.15
- new net N$1: R6.2, U2.20
- new net N$11: C17.2, IC1.1, SJ1.3
- new net N$12: C16.2, IC1.4, SJ1.1
- new net N$8: PWR+.1, SJ1.2
- new net SCK: RGB.3, U5.17
- new net SI: RGB.5, U5.13
- new net SS: RGB.2, U5.14
- net AGC: now also C7.+; no longer C7.A
- net AREF: now also C15.2; no longer C14.2
- net DTR: now also C11.1; no longer C15.2
- net GND: now also C1.1, C13.2, C14.2, C15.1, C16.1, C17.1, C18.1, C2.1, C3.1, C4.-, C5.-, C6.-, C7.-, C8.1, C9.1, IC1.2, LIPO-.1, PWR-.1, R6.1, RGB.6; no longer C1.2, C10.2, C14.1, C2.2, C3.2, C4.C, C5.C, C6.C, C7.C, Q1.2
- net MIC+: now also C19.1; no longer C8.1
- net MIC-: now also C20.2; no longer C9.2
- net N$10: now also C13.1, Q2.2; no longer Q1.3
- net N$2: now also C19.2, M1.1; no longer C8.2, U3.1
- net N$3: now also C20.1, M1.2; no longer C9.1, U3.2
- net N$6: now also C8.2; no longer C10.1
- net N$7: now also MOT-.1; no longer PAD1.1
- net N$9: now also C14.1, Q2.1; no longer Q1.1
- net RESET: now also C11.2, R8.1; no longer C15.1, R6.1
- net SP+: now also SP+.1; no longer U4.RING, U4.TIP
- net SP-: now also SP-.1; no longer U4.SLEEVE
- net VCC: now also C1.2, C18.2, C2.2, C3.2, C4.+, C5.+, C6.+, C9.2, IC1.5, LIPO+.1, MOT+.1, R8.2, RGB.1; no longer C1.1, C2.1, C3.1, C4.A, C5.A, C6.A, PAD2.1, R6.2
Routing:
- added copper zone on layer 1, net GND
- removed copper zone on layer 1, net N$4

Commit message: Schema + PCB
Parts:
- removed C13, C14: 22pf, rcl:C0805
- removed Q2: (no value), crystal:HC49UP
- added ADC0: (no value), wirepad:2,15/1,0
- added C10: 100nf, rcl:C0805
- added PROG: (no value), con-lstb:MA03-2
- added Q1: CSTCR6M00G53Z, murata-filter:CSTCR6M
- moved MOT+ 24.3 mm to (21.6, 38.1)
- moved MOT- 21.0 mm to (24.8, 38.1)
- moved T1 17.1 mm to (24.8, 34.3)
- moved RGB 15.7 mm to (36.2, 38.1), turned to 0 degrees
- moved R5 15.2 mm to (25.7, 30.2), turned to 90 degrees
- moved C18 13.7 mm to (19.7, 34.0), turned to 180 degrees
- moved C16 12.5 mm to (19.7, 32.1), turned to 180 degrees
- moved R1 12.0 mm to (47.6, 22.2)
- moved U$14 11.9 mm to (28.6, 33.0)
- moved LIPO+ 11.1 mm to (17.1, 38.1)
- moved U$13 10.8 mm to (48.3, 29.8), turned to 180 degrees
- moved R8 10.8 mm to (3.49, 25.4), turned to 180 degrees
- moved SJ1 10.3 mm to (9.53, 33.0), turned to 90 degrees
- moved IC1 10.2 mm to (15.6, 33.0), turned to 270 degrees
- moved R7 7.75 mm to (47.6, 24.8)
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Connections:
- removed net RESET: C11.2, R8.1, S2.3, S2.4, U5.29
- new net ADC0: ADC0.1, C10.1, U5.23
- new net MISO: PROG.1, U5.16
- new net RST: C11.2, PROG.5, R8.1, S2.3, S2.4, U5.29
- net GND: now also C10.2, PROG.6, Q1.2; no longer C13.2, C14.2
- net M6: now also U5.11; no longer U5.9
- net M8: now also U5.9; no longer U5.11
- net MOSI: now also PROG.4
- net N$10: now also Q1.1; no longer C13.1, Q2.2
- net N$9: now also Q1.3; no longer C14.1, Q2.1
- net SCK: now also PROG.3
- net VCC: now also PROG.2
- net VIBRATOR: now also U5.24
Routing:
- net VCC: track 0.00 -> 120.5 mm, vias 0 -> 4
- net SDA: track 0.00 -> 44.1 mm, vias 0 -> 1
- net SCL: track 0.00 -> 43.1 mm, vias 0 -> 1
- net MISO: track 0.00 -> 39.7 mm, vias 0 -> 1
- net SI: track 0.00 -> 37.0 mm
- net SCK: track 0.00 -> 35.8 mm, vias 0 -> 1
- net MOSI: track 0.00 -> 35.1 mm, vias 0 -> 1
- net SS: track 0.00 -> 31.8 mm
- net LED: track 0.00 -> 31.6 mm, vias 0 -> 2
- net M3: track 0.00 -> 30.5 mm, vias 0 -> 2
- net M4: track 0.00 -> 28.1 mm, vias 0 -> 2
- net CHG: track 0.00 -> 24.5 mm, vias 0 -> 2
- net VIBRATOR: track 0.00 -> 22.6 mm
- net REC/PLAY: track 0.00 -> 17.0 mm
- net M2: track 0.00 -> 16.6 mm, vias 0 -> 2
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- added copper zone on layer 16, net GND
Other:
- board size 50.5 x 49.5 mm -> 49.2 x 40.6 mm

Commit message: PCB
Parts:
- added B1: Button, SparkFun:TACTILE_SWITCH_SMD
- moved C9 10.5 mm to (37.1, 26.4), turned to 90 degrees
- moved C19 5.84 mm to (34.0, 7.94)
- moved C20 5.63 mm to (34.0, 9.84)
- moved C3 5.32 mm to (29.8, 23.2)
- moved R3 4.77 mm to (39.1, 7.94)
- moved R4 4.46 mm to (38.1, 12.4)
- moved C8 3.86 mm to (41.3, 4.45)
- moved C2 3.84 mm to (34.0, 14.9)
- moved M1 3.72 mm to (43.5, 10.8)
- moved R6 3.62 mm to (34.0, 11.7)
- moved R2 3.55 mm to (39.1, 4.45)
- moved C5 3.42 mm to (34.9, 17.8)
- moved R1 3.31 mm to (44.5, 21.3), turned to 270 degrees
- moved R7 3.31 mm to (44.5, 25.7), turned to 90 degrees
- moved C12 2.25 mm to (15.2, 25.7), turned to 270 degrees
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- renumbered JP1 to BL
Connections:
- net ADC0: now also B1.1, B1.2
- net GND: now also B1.3, B1.4
Routing:
- net VCC: track 120.5 -> 207.9 mm, vias 4 -> 8
- net RST: track 15.1 -> 51.6 mm, vias 0 -> 1
- net ADC0: track 6.49 -> 28.5 mm, vias 0 -> 2
- net N$3: track 0.00 -> 10.1 mm
- net N$2: track 0.00 -> 9.92 mm
- net MISO: track 39.7 -> 33.4 mm
- net LED: track 31.6 -> 37.6 mm
- net AGC: track 0.00 -> 5.64 mm
- net N$6: track 0.00 -> 5.40 mm
- net N$11: track 9.94 -> 5.56 mm
- net SCK: track 35.8 -> 33.0 mm
- net N$1: track 0.00 -> 2.74 mm
- net M4: track 28.1 -> 25.4 mm
- net MIC+: track 0.00 -> 2.29 mm
- net MIC-: track 0.00 -> 2.29 mm
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Other:
- board size 49.2 x 40.6 mm -> 47.6 x 40.6 mm
- board text added: "CHG"
- board text added: "LIPO"
- board text added: "VIB"

Commit message: Modif PCB - rev 0.5.1
Parts:
- removed S2: Reset, SparkFun:TACTILE_SWITCH_SMD
- added I2C: (no value), con-lstb:MA04-1
- added RESET: Reset, SparkFun:TACTILE_SWITCH_SMD
- moved U$14 7.89 mm to (22.9, 27.3)
- moved PROG 3.18 mm to (31.1, 33.0)
- moved M1 0.64 mm to (42.9, 10.8)
- moved R3 0.64 mm to (38.4, 7.94)
- moved C9 0.32 mm to (36.8, 26.4)
- renumbered B1 to BTN
Connections:
- net GND: now also I2C.4, RESET.1, RESET.2; no longer S2.1, S2.2
- net RST: now also RESET.3, RESET.4; no longer S2.3, S2.4
- net SCL: now also I2C.3
- net SDA: now also I2C.2
- net VCC: now also I2C.1
Routing:
- net SDA: track 44.1 -> 56.3 mm
- net SCL: track 43.1 -> 52.1 mm
- net MISO: track 33.4 -> 28.3 mm
- net RST: track 51.6 -> 48.2 mm
- net SCK: track 33.0 -> 30.1 mm
- net N$6: track 5.40 -> 6.49 mm
- net MOSI: track 33.9 -> 33.0 mm
- net N$3: track 10.1 -> 9.29 mm
- net N$2: track 9.92 -> 9.29 mm
- net VCC: track 207.9 -> 208.3 mm, vias 8 -> 9
Other:
- board text added: "LeMurmureDuSon"
- board text added: "hugo, 07/2013"
- board text added: "rev 0.5.1"
- board text added: "www.digitalspirit.org"

Commit message: PCB Version 0.6.2
Parts:
- removed M1: ELECTRET_MICROPHON-F6035AP, microphon:F6035AP
- added MIC+, MIC-: (no value), wirepad:2,15/1,0
- moved RGB 5.08 mm to (29.2, 38.1)
- moved R1 4.49 mm to (40.0, 21.9)
- moved R7 4.46 mm to (40.0, 25.4)
- moved U$13 4.45 mm to (41.6, 29.8)
- moved PROG 4.13 mm to (27.0, 33.0)
- moved C7 3.86 mm to (31.4, 3.49), turned to 270 degrees
- moved C9 3.82 mm to (34.0, 28.9), turned to 270 degrees
- moved I2C 3.81 mm to (36.8, 33.0)
- moved MOT- 3.81 mm to (19.7, 38.1)
- moved MOT+ 3.81 mm to (17.1, 38.1)
- moved C8 3.70 mm to (39.4, 7.62)
- moved R2 3.43 mm to (36.2, 6.35), turned to 180 degrees
- moved T1 3.19 mm to (21.0, 34.3)
- moved R5 3.18 mm to (21.9, 30.5)
- moved R4 2.56 mm to (35.6, 12.7)
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Connections:
- net N$2: now also MIC+.1; no longer M1.1
- net N$3: now also MIC-.1; no longer M1.2
Routing:
- net VCC: track 208.3 -> 195.5 mm
- net GND: track 0.00 -> 10.2 mm, vias 8 -> 10
- net SDA: track 56.3 -> 50.6 mm
- net M5: track 14.5 -> 19.7 mm
- net SCL: track 52.1 -> 47.4 mm
- net RST: track 48.2 -> 43.9 mm
- net SCK: track 30.1 -> 25.9 mm
- net MOSI: track 33.0 -> 29.4 mm
- net M1: track 14.8 -> 18.0 mm
- net M2: track 15.3 -> 18.2 mm
- net VIBRATOR: track 23.3 -> 20.5 mm
- net SI: track 36.2 -> 33.7 mm
- net N$2: track 9.29 -> 7.01 mm
- net MISO: track 28.3 -> 26.1 mm
- net N$3: track 9.29 -> 7.28 mm
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Other:
- board size 47.6 x 40.6 mm -> 42.2 x 40 mm
- board text added: "DRY"
- board text added: "DTR"
- board text added: "GND"
- board text added: "I2C"
- board text added: "MIC"
- board text added: "Max 5V"
- board text added: "PROG"
- board text added: "RGB"
- board text added: "RXI"
- board text added: "SCL"
- board text added: "SDA"
- board text added: "SP"
- board text added: "SPEAKER"
- board text added: "TXO"
- board text added: "VCC"
- board text added: "VIBRATOR"
- board text added: "rev 0.6.2"
- board text removed: "rev 0.5.1"

Commit message: Code + Doc + OpenScad
Parts:
- removed T1: (no value), transistor:SOT23-EBC
- added T2: (no value), transistor-neu-to92:SOT23-BEC
- R1, R5, R7: value (none) -> 4.7k
- moved R5 1.90 mm to (20.0, 30.5)
Connections:
- net GND: now also T2.E; no longer T1.E
- net N$5: now also T2.B; no longer T1.B
- net N$7: now also T2.C; no longer T1.C
Routing:
- net VIBRATOR: track 20.5 -> 19.2 mm
Other:
- board text added: "rev 0.6.x"
- board text removed: "rev 0.6.2"
Changed lines of the file:
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@@
 <text x="17.4625" y="35.56" size="1.016" layer="25">VIB</text>
 <text x="16.8275" y="24.765" size="1.016" layer="25">LeMurmureDuSon</text>
-<text x="16.8275" y="23.495" size="1.016" layer="25">rev 0.6.2</text>
+<text x="16.8275" y="23.495" size="1.016" layer="25">rev 0.6.x</text>
 <text x="31.115" y="9.8425" size="1.016" layer="26" rot="MR0">www.digitalspirit.org</text>
 <text x="31.115" y="8.255" size="1.016" layer="26" rot="MR0">hugo, 07/2013</text>
@@
 </element>
 <element name="U$14" library="SparkFun" package="OSHW-LOGO-S" value="OSHW-LOGOS" x="22.5425" y="26.9875"/>
-<element name="T1" library="transistor" package="SOT23-EBC" value="" x="20.955" y="34.29" smashed="yes">
-<attribute name="NAME" x="21.59" y="35.2425" size="0.8128" layer="25"/>
-<attribute name="VALUE" x="19.05" y="31.115" size="1.27" layer="27"/>
-</element>
-<element name="R5" library="rcl" package="M0805" value="" x="21.9075" y="30.48" smashed="yes" rot="R90">
-<attribute name="NAME" x="20.955" y="30.7975" size="0.8128" layer="25" rot="R180"/>
-<attribute name="VALUE" x="24.4475" y="29.21" size="1.27" layer="27" rot="R90"/>
+<element name="R5" library="rcl" package="M0805" value="4.7k" x="20.0025" y="30.48" smashed="yes" rot="R90">
+<attribute name="NAME" x="22.86" y="31.115" size="0.8128" layer="25" rot="R180"/>
+<attribute name="VALUE" x="22.5425" y="29.21" size="1.27" layer="27" rot="R90"/>
 </element>
 <element name="MOT-" library="wirepad" package="2,15/1,0" value="" x="19.685" y="38.1" smashed="yes">
@@
 <attribute name="VALUE" x="5.3975" y="7.62" size="1.27" layer="27" rot="R90"/>
 </element>
-<element name="R1" library="rcl" package="M0805" value="" x="40.005" y="21.9075" smashed="yes" rot="R270">
+<element name="R1" library="rcl" package="M0805" value="4.7k" x="40.005" y="21.9075" smashed="yes" rot="R270">
 <attribute name="NAME" x="39.37" y="19.05" size="0.8128" layer="25"/>
 <attribute name="VALUE" x="37.465" y="23.1775" size="1.27" layer="27" rot="R270"/>
 </element>
-<element name="R7" library="rcl" package="M0805" value="" x="40.005" y="25.4" smashed="yes" rot="R90">
+<element name="R7" library="rcl" package="M0805" value="4.7k" x="40.005" y="25.4" smashed="yes" rot="R90">
 <attribute name="NAME" x="39.37" y="27.305" size="0.8128" layer="25" rot="R180" align="top-right"/>
 <attribute name="VALUE" x="42.545" y="24.13" size="1.27" layer="27" rot="R90"/>
@@
 </element>
 <element name="C12" library="rcl" package="C0805" value="100nf" x="14.9225" y="25.7175" smashed="yes" rot="R270">
-<attribute name="NAME" x="16.1925" y="26.67" size="1.016" layer="25"/>
+<attribute name="NAME" x="13.6525" y="27.94" size="1.016" layer="25"/>
 <attribute name="VALUE" x="12.3825" y="26.9875" size="1.27" layer="27" rot="R270"/>
 </element>
@@
 <attribute name="VALUE" x="38.1" y="14.335" size="0.0254" layer="27"/>
 </element>
+<element name="T2" library="transistor-neu-to92" package="SOT23-BEC" value="" x="20.955" y="34.29"/>
 </elements>
 <signals>
@@
 <contactref element="U2" pad="8"/>
 <contactref element="U2" pad="1"/>
-<contactref element="T1" pad="E"/>
 <contactref element="U$13" pad="GND"/>
 <contactref element="RESET" pad="1"/>
@@
 <wire x1="18.1" y1="7.3" x2="18.415" y2="6.985" width="0.254" layer="1"/>
 <wire x1="18.415" y1="6.985" x2="19.177" y2="6.985" width="0.254" layer="1"/>
-<via x="17.4625" y="27.6225" extent="1-16" drill="0.6" diameter="1.016"/>
+<via x="17.145" y="27.305" extent="1-16" drill="0.6" diameter="1.016"/>
 <via x="27.305" y="2.8575" extent="1-16" drill="0.6" diameter="1.016"/>
 <wire x1="28.956" y1="5.715" x2="27.305" y2="5.715" width="0.254" layer="1"/>
@@
 </polygon>
 <wire x1="27.6225" y1="2.2225" x2="28.8925" y2="2.2225" width="0.4064" layer="1"/>
+<contactref element="T2" pad="E"/>
 </signal>
 <signal name="MIC+">
@@
 </signal>
 <signal name="N$5">
-<contactref element="T1" pad="B"/>
 <contactref element="R5" pad="2"/>
-<wire x1="21.905" y1="33.19" x2="21.905" y2="32.0675" width="0.254" layer="1"/>
-<wire x1="21.905" y1="32.0675" x2="21.9075" y2="31.43" width="0.254" layer="1"/>
+<contactref element="T2" pad="B"/>
+<wire x1="20.0025" y1="31.43" x2="20.0025" y2="33.1875" width="0.254" layer="1"/>
+<wire x1="20.0025" y1="33.1875" x2="20.005" y2="33.19" width="0.254" layer="1"/>
 </signal>
 <signal name="N$7">
-<contactref element="T1" pad="C"/>
 <contactref element="MOT-" pad="1"/>
 <wire x1="19.685" y1="38.1" x2="20.955" y2="36.83" width="0.254" layer="1"/>
+<contactref element="T2" pad="C"/>
 <wire x1="20.955" y1="36.83" x2="20.955" y2="35.39" width="0.254" layer="1"/>
 </signal>
@@
 <wire x1="14.2875" y1="19.685" x2="14.9225" y2="20.32" width="0.254" layer="1"/>
 <wire x1="14.9225" y1="20.32" x2="14.9225" y2="21.2725" width="0.254" layer="1"/>
-<wire x1="21.905" y1="29.845" x2="21.9075" y2="29.53" width="0.254" layer="1"/>
 <wire x1="8.3125" y1="20.8026" x2="8.3125" y2="19.945" width="0.254" layer="1"/>
 <wire x1="8.3125" y1="19.945" x2="8.5725" y2="19.685" width="0.254" layer="1"/>
@@
 <wire x1="14.9225" y1="21.2725" x2="15.5575" y2="21.9075" width="0.254" layer="1"/>
 <wire x1="15.5575" y1="21.9075" x2="15.5575" y2="22.70125" width="0.254" layer="1"/>
-<wire x1="15.5575" y1="22.70125" x2="20.79625" y2="27.94" width="0.254" layer="1"/>
-<wire x1="20.79625" y1="27.94" x2="21.2725" y2="27.94" width="0.254" layer="1"/>
-<wire x1="21.2725" y1="27.94" x2="21.9075" y2="28.575" width="0.254" layer="1"/>
-<wire x1="21.9075" y1="28.575" x2="21.9075" y2="29.53" width="0.254" layer="1"/>
+<wire x1="15.5575" y1="22.70125" x2="20.0025" y2="27.14625" width="0.254" layer="1"/>
+<wire x1="20.0025" y1="27.14625" x2="20.0025" y2="29.53" width="0.254" layer="1"/>
 </signal>
 <signal name="SDA">
@@
 <wire x1="13.9125" y1="20.8026" x2="13.9125" y2="20.8975" width="0.254" layer="1"/>
 <wire x1="13.9125" y1="20.8975" x2="13.97" y2="20.955" width="0.254" layer="1"/>
-<wire x1="19.3675" y1="28.2575" x2="20.0025" y2="28.8925" width="0.254" layer="16"/>
+<wire x1="18.7325" y1="27.6225" x2="20.0025" y2="28.8925" width="0.254" layer="16"/>
 <wire x1="20.0025" y1="28.8925" x2="24.765" y2="28.8925" width="0.254" layer="16"/>
 <wire x1="24.765" y1="28.8925" x2="25.7175" y2="29.845" width="0.254" layer="16"/>
-<via x="19.3675" y="28.2575" extent="1-16" drill="0.6" diameter="1.016"/>
+<via x="18.7325" y="27.6225" extent="1-16" drill="0.6" diameter="1.016"/>
 <wire x1="13.97" y1="20.955" x2="13.97" y2="21.2725" width="0.254" layer="1"/>
 <wire x1="13.97" y1="21.2725" x2="14.9225" y2="22.225" width="0.254" layer="1"/>
 <wire x1="14.9225" y1="22.225" x2="14.9225" y2="23.01875" width="0.254" layer="1"/>
-<wire x1="14.9225" y1="23.01875" x2="19.3675" y2="27.46375" width="0.254" layer="1"/>
-<wire x1="19.3675" y1="27.46375" x2="19.3675" y2="28.2575" width="0.254" layer="1"/>
+<wire x1="14.9225" y1="23.01875" x2="18.7325" y2="26.82875" width="0.254" layer="1"/>
+<wire x1="18.7325" y1="26.82875" x2="18.7325" y2="27.6225" width="0.254" layer="1"/>
 <wire x1="27.94" y1="38.1" x2="27.94" y2="36.195" width="0.254" layer="1"/>
 <wire x1="27.94" y1="36.195" x2="26.9875" y2="35.2425" width="0.254" layer="1"/>
