File: pcb/mds.brd (EAGLE design)
At the start: 42.2 x 40 mm, 62 parts, among them IC1 MAX1555, Q2 MOSFET-P, U2 ISD1900ISD1932, U3 ADXL345, U5 ATMEGA328

Commit message: Update CAD
Parts:
- removed D4: (no value), OPL Eagle Library:LL-34
- added D1: 1N4148, OPL Eagle Library:LL-34
- added R16: 33k, rcl:M0805
- added R17: 2.2k, rcl:M0805
- added T1: (no value), transistor-neu-to92:SOT23-BEC
- D3: value (none) -> Schottky
- R10: value 4.7k -> 1.2M
- moved LDR+ 115.3 mm to (41.9, 47.0)
- moved LDR- 110.9 mm to (36.8, 47.9)
- moved R15 98.0 mm to (29.8, 46.7)
- moved D3 87.6 mm to (21.9, 46.0)
- moved Q2 80.6 mm to (14.6, 44.8)
- moved R10 73.9 mm to (8.57, 45.1)
Connections:
- new net N$4: R16.1, T1.B
- new net PWR_STATUS: D1.A, U5.1
- net CHG: now also D1.C; no longer U5.1
- net GND: now also R17.2, T1.E
- net N$9: now also Q2.1, R10.1, T1.C; no longer D4.C
- net PWR_CMD: now also R16.2, R17.1; no longer D3.A, D4.A, Q2.1, R10.1
Routing:
- net CHG: track 41.8 -> 40.3 mm
Changed lines of the file:
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@@
 <?xml version="1.0" encoding="utf-8"?>
 <!DOCTYPE eagle SYSTEM "eagle.dtd">
-<eagle version="6.5.0">
+<eagle version="7.3.0">
 <drawing>
 <settings>
@@
 <pass name="Default">
 <param name="RoutingGrid" value="50mil"/>
+<param name="AutoGrid" value="1"/>
+<param name="Efforts" value="0"/>
+<param name="TopRouterVariant" value="1"/>
 <param name="tpViaShape" value="round"/>
 <param name="PrefDir.1" value="|"/>
@@
 <attribute name="OC_FARNELL" value="unknown" x="31.75" y="38.1" size="1.778" layer="27" display="off"/>
 </element>
-<element name="R10" library="rcl" package="M0805" value="4.7k" x="2.2225" y="-28.575"/>
-<element name="Q2" library="OPL Eagle Library" package="SOT23" value="MOSFET-P" x="2.54" y="-34.925"/>
-<element name="D3" library="OPL Eagle Library" package="LL-34" value="" x="2.54" y="-39.37"/>
-<element name="D4" library="OPL Eagle Library" package="LL-34" value="" x="2.54" y="-43.18"/>
+<element name="R10" library="rcl" package="M0805" value="1.2M" x="8.5725" y="45.085"/>
+<element name="Q2" library="OPL Eagle Library" package="SOT23" value="MOSFET-P" x="14.605" y="44.7675"/>
+<element name="D3" library="OPL Eagle Library" package="LL-34" value="Schottky" x="21.9075" y="46.0375"/>
 <element name="U3" library="SparkFun-Sensors" package="LGA14" value="ADXL345" x="9.8425" y="4.445"/>
 <element name="U$1" library="SparkFun-Sensors" package="16LPCC" value="HMC5883LSMD" x="14.9225" y="6.0325"/>
-<element name="R15" library="rcl" package="M0805" value="4.7k" x="2.2225" y="-47.3075"/>
-<element name="LDR-" library="wirepad" package="1,6/0,8" value="" x="1.27" y="-57.15"/>
-<element name="LDR+" library="wirepad" package="1,6/0,8" value="" x="1.27" y="-60.96"/>
+<element name="R15" library="rcl" package="M0805" value="4.7k" x="29.845" y="46.6725"/>
+<element name="LDR-" library="wirepad" package="1,6/0,8" value="" x="36.83" y="47.9425"/>
+<element name="LDR+" library="wirepad" package="1,6/0,8" value="" x="41.91" y="46.99"/>
+<element name="T1" library="transistor-neu-to92" package="SOT23-BEC" value="" x="17.145" y="49.2125"/>
+<element name="R16" library="rcl" package="M0805" value="33k" x="26.035" y="42.545"/>
+<element name="R17" library="rcl" package="M0805" value="2.2k" x="34.6075" y="43.815"/>
+<element name="D1" library="OPL Eagle Library" package="LL-34" value="1N4148" x="2.54" y="-2.54"/>
 </elements>
 <signals>
@@
 <contactref element="U$1" pad="11"/>
 <contactref element="R15" pad="1"/>
-<wire x1="40.64" y1="33.02" x2="39.6875" y2="37.465" width="0" layer="19" extent="1-1"/>
+<contactref element="T1" pad="E"/>
+<contactref element="R17" pad="2"/>
+<wire x1="34.29" y1="38.1" x2="35.5575" y2="43.815" width="0" layer="19" extent="1-1"/>
 <wire x1="16.2925" y1="6.2825" x2="17.145" y2="7.3" width="0" layer="19" extent="1-1"/>
 <wire x1="16.2925" y1="5.2825" x2="16.2925" y2="6.2825" width="0" layer="19" extent="1-1"/>
+<wire x1="39.6875" y1="37.465" x2="40.64" y2="33.02" width="0" layer="19" extent="1-1"/>
 <wire x1="2.54" y1="2.54" x2="8.6425" y2="5.545" width="0" layer="19" extent="1-1"/>
-<wire x1="1.2725" y1="-47.3075" x2="2.54" y2="2.54" width="0" layer="19" extent="1-1"/>
+<wire x1="28.895" y1="46.6725" x2="35.5575" y2="43.815" width="0" layer="19" extent="1-1"/>
+<wire x1="18.095" y1="48.1125" x2="13.97" y2="38.1" width="0" layer="19" extent="1-1"/>
 </signal>
 <signal name="MIC+">
@@
 <contactref element="U$1" pad="4"/>
 <contactref element="LDR+" pad="1"/>
-<wire x1="32.385" y1="36.195" x2="29.21" y2="38.1" width="0" layer="19" extent="16-16"/>
+<wire x1="32.385" y1="36.195" x2="41.91" y2="46.99" width="0" layer="19" extent="16-16"/>
 <wire x1="15.6725" y1="7.4025" x2="17.145" y2="5.4" width="0" layer="19" extent="1-1"/>
 <wire x1="13.5525" y1="6.2825" x2="15.6725" y2="7.4025" width="0" layer="19" extent="1-1"/>
@@
 <wire x1="11.8425" y1="5.545" x2="13.5525" y2="5.2825" width="0" layer="19" extent="1-1"/>
 <wire x1="11.90625" y1="8.41375" x2="13.5525" y2="6.2825" width="0" layer="19" extent="1-1"/>
+<wire x1="29.21" y1="38.1" x2="32.385" y2="36.195" width="0" layer="19" extent="16-16"/>
 <wire x1="7.8425" y1="5.545" x2="11.8425" y2="5.545" width="0" layer="19" extent="1-1"/>
-<wire x1="3.1725" y1="-28.575" x2="7.8425" y2="5.545" width="0" layer="19" extent="1-1"/>
-<wire x1="2.54" y1="-33.909" x2="3.1725" y2="-28.575" width="0" layer="19" extent="1-1"/>
-<wire x1="1.27" y1="-60.96" x2="2.54" y2="-33.909" width="0" layer="19" extent="1-1"/>
+<wire x1="14.605" y1="45.7835" x2="19.05" y2="38.1" width="0" layer="19" extent="1-1"/>
+<wire x1="9.5225" y1="45.085" x2="14.605" y2="45.7835" width="0" layer="19" extent="1-1"/>
 </signal>
 <signal name="N$5">
@@
 <signal name="CHG">
 <contactref element="IC1" pad="3"/>
-<contactref element="U5" pad="1"/>
 <wire x1="12.035" y1="32.07" x2="12.0625" y2="32.07" width="0.254" layer="1"/>
 <wire x1="12.0625" y1="32.07" x2="10.795" y2="32.0675" width="0.254" layer="1"/>
@@
 <wire x1="10.795" y1="32.0675" x2="8.89" y2="32.0675" width="0.254" layer="16"/>
 <wire x1="8.89" y1="32.0675" x2="7.9375" y2="31.115" width="0.254" layer="16"/>
-<wire x1="7.9375" y1="31.115" x2="7.9375" y2="28.8925" width="0.254" layer="16"/>
-<via x="7.9375" y="28.8925" extent="1-16" drill="0.6"/>
-<wire x1="7.9375" y1="28.8925" x2="6.665" y2="28.575" width="0.254" layer="1"/>
-<wire x1="7.9375" y1="28.8925" x2="6.6675" y2="28.8925" width="0.254" layer="1"/>
-<wire x1="6.6675" y1="28.8925" x2="6.6675" y2="27.6225" width="0.254" layer="1"/>
+<wire x1="7.9375" y1="31.115" x2="7.9375" y2="28.575" width="0.254" layer="16"/>
+<via x="7.9375" y="28.575" extent="1-16" drill="0.6"/>
+<wire x1="6.6675" y1="28.575" x2="6.665" y2="28.575" width="0.254" layer="1"/>
+<wire x1="7.9375" y1="28.575" x2="6.6675" y2="28.575" width="0.254" layer="1"/>
+<wire x1="6.6675" y1="28.575" x2="6.6675" y2="27.6225" width="0.254" layer="1"/>
 <wire x1="6.6675" y1="27.6225" x2="6.35" y2="27.305" width="0.254" layer="1"/>
 <wire x1="6.35" y1="27.305" x2="1.27" y2="27.305" width="0.254" layer="1"/>
@@
 <wire x1="1.27" y1="9.525" x2="6.19125" y2="9.525" width="0.254" layer="1"/>
 <wire x1="6.19125" y1="9.525" x2="6.5151" y2="9.20115" width="0.254" layer="1"/>
-<wire x1="8.3125" y1="9.6774" x2="8.09625" y2="9.68375" width="0.254" layer="1"/>
 <wire x1="8.09625" y1="9.68375" x2="7.77875" y2="9.68375" width="0.254" layer="1"/>
 <wire x1="7.77875" y1="9.68375" x2="7.29615" y2="9.20115" width="0.254" layer="1"/>
 <wire x1="7.29615" y1="9.20115" x2="6.5151" y2="9.20115" width="0.254" layer="1"/>
 <contactref element="D3" pad="C"/>
-<wire x1="6.5151" y1="9.20115" x2="4.064" y2="-39.37" width="0" layer="19" extent="1-1"/>
+<contactref element="D1" pad="C"/>
+<wire x1="12.0625" y1="32.07" x2="23.4315" y2="46.0375" width="0" layer="19" extent="1-1"/>
+<wire x1="4.064" y1="-2.54" x2="6.5151" y2="9.20115" width="0" layer="19" extent="1-1"/>
 </signal>
 <signal name="MISO">
@@
 <signal name="PWR_CMD">
 <contactref element="U5" pad="13"/>
-<contactref element="R10" pad="1"/>
-<contactref element="Q2" pad="1"/>
-<contactref element="D4" pad="A"/>
-<contactref element="D3" pad="A"/>
-<wire x1="1.016" y1="-39.37" x2="1.016" y2="-43.18" width="0" layer="19" extent="1-1"/>
-<wire x1="1.651" y1="-35.941" x2="1.016" y2="-39.37" width="0" layer="19" extent="1-1"/>
-<wire x1="1.2725" y1="-28.575" x2="1.651" y2="-35.941" width="0" layer="19" extent="1-1"/>
-<wire x1="15.4051" y1="14.37" x2="1.2725" y2="-28.575" width="0" layer="19" extent="1-1"/>
+<contactref element="R16" pad="2"/>
+<contactref element="R17" pad="1"/>
+<wire x1="26.985" y1="42.545" x2="33.6575" y2="43.815" width="0" layer="19" extent="1-1"/>
+<wire x1="15.4051" y1="14.37" x2="26.985" y2="42.545" width="0" layer="19" extent="1-1"/>
 </signal>
 <signal name="+UB">
 <contactref element="Q2" pad="2"/>
 <contactref element="LIPO+" pad="1"/>
-<wire x1="3.429" y1="-35.941" x2="15.875" y2="38.1" width="0" layer="19" extent="1-1"/>
-</signal>
-<signal name="N$9">
-<contactref element="D4" pad="C"/>
+<wire x1="15.875" y1="38.1" x2="15.494" y2="43.7515" width="0" layer="19" extent="1-1"/>
 </signal>
 <signal name="AD_INT1">
@@
 <contactref element="LDR-" pad="1"/>
 <contactref element="R15" pad="2"/>
-<wire x1="3.1725" y1="-47.3075" x2="1.27" y2="-57.15" width="0" layer="19" extent="1-1"/>
+<wire x1="30.795" y1="46.6725" x2="36.83" y2="47.9425" width="0" layer="19" extent="1-1"/>
+</signal>
+<signal name="N$4">
+<contactref element="T1" pad="B"/>
+<contactref element="R16" pad="1"/>
+<wire x1="16.195" y1="48.1125" x2="25.085" y2="42.545" width="0" layer="19" extent="1-1"/>
+</signal>
+<signal name="PWR_STATUS">
+<contactref element="D1" pad="A"/>
+<contactref element="U5" pad="1"/>
+<wire x1="1.016" y1="-2.54" x2="8.3125" y2="9.6774" width="0" layer="19" extent="1-1"/>
+</signal>
+<signal name="N$9">
+<contactref element="T1" pad="C"/>
+<contactref element="R10" pad="1"/>
+<contactref element="Q2" pad="1"/>
+<wire x1="13.716" y1="43.7515" x2="17.145" y2="50.3125" width="0" layer="19" extent="1-1"/>
+<wire x1="7.6225" y1="45.085" x2="13.716" y2="43.7515" width="0" layer="19" extent="1-1"/>
 </signal>
 </signals>
