File: pcb/mds.sch (EAGLE design)
At the start: 27 parts, among them U2 ISD1900ISD1932, U3 MICELECTRET_SMD, U4 AUDIO-JACK2SMD

Commit message: Electronique
Parts:
- removed JP4, JP5, JP8: (no value), SparkFun:M02PTH
- removed JP7: (no value), SparkFun:M08
- removed JP9: (no value), SparkFun:M06SIP
- removed S1: (no value), SparkFun:SWITCH-SPSTSMD
- removed U$10: ARDUINOMICRO, adafruit:ARDUINOMICRO
- added U$15: ARDUINO_MINI, SparkFun-Boards:ARDUINO_MINI
Connections:
- removed net E0: JP7.8, U2.E0/_M5
- removed net E1: JP7.7, U2.E1/_M6
- removed net E2: JP7.6, U2.E2/_M7
- removed net E3: JP7.5, U2.E3/_M8
- removed net FMC1: JP9.6, U2._PLAYL/FMC1
- removed net FMC2: JP9.5, U2._PLAYE/FMC2
- removed net MODE: S1.P, U2.ADDR/_DRCT
- removed net REC: JP9.4, U2._REC
- removed net S0: JP7.4, U2.S0/_M1
- removed net S1: JP7.3, U2.S1/_M2
- removed net S2: JP7.2, U2.S2/_M3
- removed net S3: JP7.1, U2.S3/_M4
- net 5V: no longer JP4.2, S1.S
- net AGC: no longer JP9.2
- net FT: no longer JP9.1
- net GND: now also U2.ADDR/_DRCT; no longer JP4.1, S1.O
- net LED: no longer JP8.1
- net ROSC: no longer JP9.3
- net SP+: no longer JP5.1
- net SP-: no longer JP5.2
- net XCLK: no longer JP8.2
Other:
- note added: "Core"
- note added: "Interface"
- note added: "Power"
- note added: "Sensor"
- note added: "Sound"
- moved on the sheet: C1, C10, C2, C3, C4, C5, C6, C7, C8, C9, LED1, R1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

Commit message: Schema development
Parts:
- removed LED1: Red, SparkFun:LED0603
- removed U$15: ARDUINO_MINI, SparkFun-Boards:ARDUINO_MINI
- added C12, C14, C15: 0.1uF, SparkFun:CAP0402-CAP
- added JP1: FTDI Basic, SparkFun:ARDUINO_SERIAL_PROGRAMPTH
- added JP8: FIDUCIALUFIDUCIAL, SparkFun:FIDUCIALUFIDUCIAL
- added PAD1, PAD2: (no value), wirepad:2,15/1,0
- added Q1: 8/16/20MHz, SparkFun:RESONATORSMD
- added R5, R7: (no value), rcl:R-EU_M0805
- added R6: 10K, SparkFun:RESISTOR0402-RES
- added S2: Reset, SparkFun:TAC_SWITCHSMD
- added T1: (no value), transistor:-NPN-SOT23-EBC
- added U5: ATMEGA328, SparkFun:ATMEGA168
- R1: value 1k -> (none); device SparkFun:RESISTOR0603-RES -> rcl:R-EU_M0805
Connections:
- removed net 5V: C1.1, C2.1, C3.1, C4.+, C5.+, C6.+, LED1.A, R2.2, U2.VCCA, U2.VCCD, U2.VCCP
- removed net N$1: LED1.C, R1.2
- removed net XCLK: U2.XCLK/FMC3
- new net AREF: C14.2, U5.AREF
- new net DTR: C15.2, JP1.DTR
- new net M1: U2.S0/_M1, U5.PC2(ADC2)
- new net M2: U2.S1/_M2, U5.PC3(ADC3)
- new net M3: U2.S2/_M3, U5.ADC6
- new net M4: U2.S3/_M4, U5.ADC7
- new net M5: U2.E0/_M5, U5.PD4(XCK/T0)
- new net M6: U2.E1/_M6, U5.PD5(T1)
- new net M7: U2.E2/_M7, U5.PD6(AIN0)
- new net M8: U2.E3/_M8, U5.PD7(AIN1)
- new net N$10: Q1.3, U5.PB6(XTAL1/TOSC1)
- new net N$5: R5.2, T1.B
- new net N$7: PAD1.P, T1.C
- new net N$9: Q1.1, U5.PB7(XTAL2/TOSC2)
- new net REC/PLAY: U2._REC, U5.PB0(ICP)
- new net RESET: C15.1, R6.1, S2.3, S2.4, U5.PC6(/RESET)
- new net RXI: JP1.TXO, U5.PD0(RXD)
- new net SCL: R7.1, U$13.SCL, U5.PC5(ADC5/SCL)
- new net SDA: R1.1, U$13.SDA, U5.PC4(ADC4/SDA)
- new net TXO: JP1.RXI, U5.PD1(TXD)
- new net VCC: C1.1, C12.2, C2.1, C3.1, C4.+, C5.+, C6.+, JP1.VCC, PAD2.P, R1.2, R2.2, R6.2, R7.2, U$13.VCC, U2.VCCA, U2.VCCD, U2.VCCP, U2.XCLK/FMC3, U2._PLAYE/FMC2, U2._PLAYL/FMC1, U5.AVCC, U5.VCC@1, U5.VCC@2
- new net VIBRATOR: R5.1
- net GND: now also C12.1, C14.1, JP1.CTS, JP1.GND, Q1.2, S2.1, S2.2, T1.E, U$13.GND, U5.AGND, U5.GND@1, U5.GND@2
- net LED: now also U5.PD2(INT0); no longer R1.1
Other:
- moved on the sheet: C1, C2, C3, C4, C5, C6

Commit message: Schema + PCB
Parts:
- removed C10: 4.7uF, SparkFun:CAP0603-CAP
- removed JP8: FIDUCIALUFIDUCIAL, SparkFun:FIDUCIALUFIDUCIAL
- removed PAD1, PAD2: (no value), wirepad:2,15/1,0
- removed Q1: 8/16/20MHz, SparkFun:RESONATORSMD
- removed U3: MICELECTRET_SMD, SparkFun:MICELECTRET_SMD
- removed U4: AUDIO-JACK2SMD, SparkFun:AUDIO-JACK2SMD
- added C11, C16, C17, C18, C19, C20: 100nf, rcl:C-EUC0805
- added C13: 22pf, rcl:C-EUC0805
- added IC1: MAX1555, maxim:MAX1555
- added LIPO+, LIPO-, MOT+, MOT-, PWR+, PWR-, SP+, SP-: (no value), wirepad:2,15/1,0
- added M1: ELECTRET_MICROPHON-F6035AP, microphon:ELECTRET_MICROPHON-F6035AP
- added Q2: (no value), crystal:CRYSTALHC49UP
- added R8: 10k, rcl:R-EU_M0805
- added RGB: (no value), con-lstb:MA06-1
- added SJ1: (no value), jumper:SJ2W
- C1, C2, C3, C8, C9: value 0.1uF -> 100nf; device SparkFun:CAP0603-CAP -> rcl:C-EUC0805
- C12, C15: value 0.1uF -> 100nf; device SparkFun:CAP0402-CAP -> rcl:C-EUC0805
- C14: value 0.1uF -> 22pf; device SparkFun:CAP0402-CAP -> rcl:C-EUC0805
- C4, C5, C6, C7: value 10uF -> 10uf; device SparkFun:CAP_POL1206 -> rcl:CPOL-EUCT3528
- R2, R3, R4: device SparkFun:RESISTOR0603-RES -> rcl:R-EU_M0805
- R6: value 10K -> (none); device SparkFun:RESISTOR0402-RES -> rcl:R-EU_M0805
Connections:
- removed net ROSC: U2.ROSC
- new net CHG: IC1.!CHG, U5.PD3(INT1)
- new net MOSI: RGB.4, U5.PB3(MOSI/OC2)
- new net N$1: R6.2, U2.ROSC
- new net N$11: C17.2, IC1.USB, SJ1.3
- new net N$12: C16.2, IC1.DC, SJ1.1
- new net N$8: PWR+.P, SJ1.2
- new net SCK: RGB.3, U5.PB5(SCK)
- new net SI: RGB.5, U5.PB1(OC1A)
- new net SS: RGB.2, U5.PB2(SS/OC1B)
- net AREF: now also C15.2; no longer C14.2
- net DTR: now also C11.1; no longer C15.2
- net GND: now also C1.1, C13.2, C14.2, C15.1, C16.1, C17.1, C18.1, C2.1, C3.1, C8.1, C9.1, IC1.GND, LIPO-.P, PWR-.P, R6.1, RGB.6; no longer C1.2, C10.2, C14.1, C2.2, C3.2, Q1.2
- net MIC+: now also C19.1; no longer C8.1
- net MIC-: now also C20.2; no longer C9.2
- net N$10: now also C13.1, Q2.2; no longer Q1.3
- net N$2: now also C19.2, M1.1; no longer C8.2, U3.1
- net N$3: now also C20.1, M1.2; no longer C9.1, U3.2
- net N$6: now also C8.2; no longer C10.1
- net N$7: now also MOT-.P; no longer PAD1.P
- net N$9: now also C14.1, Q2.1; no longer Q1.1
- net RESET: now also C11.2, R8.1; no longer C15.1, R6.1
- net SP+: now also SP+.P; no longer U4.RING, U4.TIP
- net SP-: now also SP-.P; no longer U4.SLEEVE
- net VCC: now also C1.2, C18.2, C2.2, C3.2, C9.2, IC1.BAT, LIPO+.P, MOT+.P, R8.2, RGB.1; no longer C1.1, C2.1, C3.1, PAD2.P, R6.2
Other:
- moved on the sheet: C1, C14, C15, C2, C3, C4, C5, C6, C7, C8, C9, R5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

Commit message: Schema + PCB
Parts:
- removed C13, C14: 22pf, rcl:C-EUC0805
- removed Q2: (no value), crystal:CRYSTALHC49UP
- added ADC0: (no value), wirepad:2,15/1,0
- added C10: 100nf, rcl:C-EUC0805
- added PROG: (no value), con-lstb:MA03-2
- added Q1: CSTCR6M00G53Z, murata-filter:CSTCR6M00G53Z
Connections:
- removed net RESET: C11.2, R8.1, S2.3, S2.4, U5.PC6(/RESET)
- new net ADC0: ADC0.P, C10.1, U5.PC0(ADC0)
- new net MISO: PROG.1, U5.PB4(MISO)
- new net RST: C11.2, PROG.5, R8.1, S2.3, S2.4, U5.PC6(/RESET)
- net GND: now also C10.2, PROG.6, Q1.2; no longer C13.2, C14.2
- net M6: now also U5.PD7(AIN1); no longer U5.PD5(T1)
- net M8: now also U5.PD5(T1); no longer U5.PD7(AIN1)
- net MOSI: now also PROG.4
- net N$10: now also Q1.1; no longer C13.1, Q2.2
- net N$9: now also Q1.3; no longer C14.1, Q2.1
- net SCK: now also PROG.3
- net VCC: now also PROG.2
- net VIBRATOR: now also U5.PC1(ADC1)

Commit message: PCB
Parts:
- added B1: Button, SparkFun:TAC_SWITCHSMD
- renumbered JP1 to BL
Connections:
- net ADC0: now also B1.1, B1.2
- net GND: now also B1.3, B1.4
Other:
- moved on the sheet: ADC0
Changed lines of the file:
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@@
 <setting verticaltext="up"/>
 </settings>
-<grid distance="0.1" unitdist="inch" unit="inch" style="lines" multiple="1" display="no" altdistance="0.01" altunitdist="inch" altunit="inch"/>
+<grid distance="0.1" unitdist="inch" unit="inch" style="dots" multiple="1" display="yes" altdistance="0.01" altunitdist="inch" altunit="inch"/>
 <layers>
 <layer number="1" name="Top" color="4" fill="1" visible="no" active="no"/>
@@
 <part name="U5" library="SparkFun" deviceset="ATMEGA168" device="" value="ATMEGA328"/>
 <part name="GND19" library="SparkFun" deviceset="GND" device=""/>
-<part name="JP1" library="SparkFun" deviceset="ARDUINO_SERIAL_PROGRAM" device="PTH" value="FTDI Basic"/>
+<part name="BL" library="SparkFun" deviceset="ARDUINO_SERIAL_PROGRAM" device="PTH" value="FTDI Basic"/>
 <part name="P+12" library="supply1" deviceset="VCC" device=""/>
 <part name="P+14" library="supply1" deviceset="VCC" device=""/>
@@
 <part name="GND26" library="SparkFun" deviceset="GND" device=""/>
 <part name="Q1" library="murata-filter" deviceset="CSTCR" device="" technology="6M00G53Z"/>
+<part name="B1" library="SparkFun" deviceset="TAC_SWITCH" device="SMD" value="Button"/>
+<part name="GND27" library="SparkFun" deviceset="GND" device=""/>
 </parts>
 <sheets>
@@
 </instance>
 <instance part="GND19" gate="1" x="58.42" y="45.72"/>
-<instance part="JP1" gate="G$1" x="22.86" y="22.86"/>
+<instance part="BL" gate="G$1" x="22.86" y="22.86"/>
 <instance part="P+12" gate="VCC" x="233.68" y="83.82" smashed="yes">
 <attribute name="VALUE" x="231.14" y="83.82" size="1.778" layer="96" rot="R180"/>
@@
 <instance part="PROG" gate="1" x="106.68" y="22.86" rot="R180"/>
 <instance part="RGB" gate="1" x="360.68" y="205.74" rot="R180"/>
-<instance part="ADC0" gate="1" x="314.96" y="180.34" smashed="yes" rot="R180">
-<attribute name="NAME" x="323.723" y="181.0258" size="1.778" layer="95" rot="R180"/>
-<attribute name="VALUE" x="316.103" y="183.642" size="1.778" layer="96" rot="R180"/>
+<instance part="ADC0" gate="1" x="325.12" y="185.42" smashed="yes" rot="R180">
+<attribute name="NAME" x="333.883" y="186.1058" size="1.778" layer="95" rot="R180"/>
+<attribute name="VALUE" x="326.263" y="188.722" size="1.778" layer="96" rot="R180"/>
 </instance>
 <instance part="C10" gate="G$1" x="129.54" y="101.6"/>
 <instance part="GND26" gate="1" x="129.54" y="91.44"/>
 <instance part="Q1" gate="G$1" x="50.8" y="78.74" rot="R270"/>
+<instance part="B1" gate="S" x="327.66" y="172.72" smashed="yes">
+<attribute name="NAME" x="330.962" y="178.054" size="1.778" layer="95" rot="R270"/>
+<attribute name="VALUE" x="324.104" y="168.148" size="1.778" layer="96"/>
+</instance>
+<instance part="GND27" gate="1" x="335.28" y="165.1"/>
 </instances>
 <busses>
@@
 <wire x1="27.94" y1="27.94" x2="35.56" y2="27.94" width="0.1524" layer="91"/>
 <label x="30.48" y="27.94" size="1.778" layer="95"/>
-<pinref part="JP1" gate="G$1" pin="CTS"/>
+<pinref part="BL" gate="G$1" pin="CTS"/>
 </segment>
 <segment>
 <wire x1="27.94" y1="30.48" x2="35.56" y2="30.48" width="0.1524" layer="91"/>
 <label x="30.48" y="30.48" size="1.778" layer="95"/>
-<pinref part="JP1" gate="G$1" pin="GND"/>
+<pinref part="BL" gate="G$1" pin="GND"/>
 </segment>
 <segment>
@@
 <junction x="116.84" y="20.32"/>
 <label x="123.19" y="21.59" size="1.778" layer="95" rot="R180"/>
+</segment>
+<segment>
+<pinref part="B1" gate="S" pin="4"/>
+<wire x1="332.74" y1="170.18" x2="335.28" y2="170.18" width="0.1524" layer="91"/>
+<wire x1="335.28" y1="170.18" x2="335.28" y2="172.72" width="0.1524" layer="91"/>
+<pinref part="B1" gate="S" pin="3"/>
+<wire x1="335.28" y1="172.72" x2="332.74" y2="172.72" width="0.1524" layer="91"/>
+<pinref part="GND27" gate="1" pin="GND"/>
+<wire x1="335.28" y1="170.18" x2="335.28" y2="167.64" width="0.1524" layer="91"/>
+<junction x="335.28" y="170.18"/>
 </segment>
 </net>
@@
 <wire x1="27.94" y1="25.4" x2="35.56" y2="25.4" width="0.1524" layer="91"/>
 <label x="30.48" y="25.4" size="1.778" layer="95"/>
-<pinref part="JP1" gate="G$1" pin="VCC"/>
+<pinref part="BL" gate="G$1" pin="VCC"/>
 </segment>
 <segment>
@@
 <wire x1="27.94" y1="20.32" x2="35.56" y2="20.32" width="0.1524" layer="91"/>
 <label x="30.48" y="20.32" size="1.778" layer="95"/>
-<pinref part="JP1" gate="G$1" pin="RXI"/>
+<pinref part="BL" gate="G$1" pin="RXI"/>
 </segment>
 </net>
@@
 <wire x1="27.94" y1="17.78" x2="35.56" y2="17.78" width="0.1524" layer="91"/>
 <label x="30.48" y="17.78" size="1.778" layer="95"/>
-<pinref part="JP1" gate="G$1" pin="DTR"/>
+<pinref part="BL" gate="G$1" pin="DTR"/>
 </segment>
 <segment>
@@
 <wire x1="27.94" y1="22.86" x2="35.56" y2="22.86" width="0.1524" layer="91"/>
 <label x="30.48" y="22.86" size="1.778" layer="95"/>
-<pinref part="JP1" gate="G$1" pin="TXO"/>
+<pinref part="BL" gate="G$1" pin="TXO"/>
 </segment>
 <segment>
@@
 <segment>
 <pinref part="ADC0" gate="1" pin="P"/>
-<wire x1="312.42" y1="180.34" x2="309.88" y2="180.34" width="0.1524" layer="91"/>
-<junction x="309.88" y="180.34"/>
-<label x="302.26" y="180.34" size="1.778" layer="95"/>
-</segment>
-</net>
+<wire x1="322.58" y1="185.42" x2="320.04" y2="185.42" width="0.1524" layer="91"/>
+<junction x="320.04" y="185.42"/>
+<label x="312.42" y="185.42" size="1.778" layer="95"/>
+</segment>
+<segment>
+<pinref part="B1" gate="S" pin="2"/>
+<wire x1="322.58" y1="170.18" x2="320.04" y2="170.18" width="0.1524" layer="91"/>
+<wire x1="320.04" y1="170.18" x2="320.04" y2="172.72" width="0.1524" layer="91"/>
+<pinref part="B1" gate="S" pin="1"/>
+<wire x1="320.04" y1="172.72" x2="322.58" y2="172.72" width="0.1524" layer="91"/>
+<wire x1="320.04" y1="170.18" x2="317.5" y2="170.18" width="0.1524" layer="91"/>
+<junction x="320.04" y="170.18"/>
+<junction x="317.5" y="170.18"/>
+<label x="307.34" y="170.18" size="1.778" layer="95"/>
+</segment>
+</net>

Commit message: Modif PCB - rev 0.5.1
Parts:
- added I2C: (no value), con-lstb:MA04-1
- renumbered B1 to BTN, S2 to RESET
Connections:
- net GND: now also I2C.4
- net SCL: now also I2C.3
- net SDA: now also I2C.2
- net VCC: now also I2C.1
Changed lines of the file:
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@@
 <part name="P+9" library="supply1" deviceset="VCC" device=""/>
 <part name="P+11" library="supply1" deviceset="VCC" device=""/>
-<part name="S2" library="SparkFun" deviceset="TAC_SWITCH" device="SMD" value="Reset"/>
+<part name="RESET" library="SparkFun" deviceset="TAC_SWITCH" device="SMD" value="Reset"/>
 <part name="GND14" library="SparkFun" deviceset="GND" device=""/>
 <part name="GND15" library="SparkFun" deviceset="GND" device=""/>
@@
 <part name="GND26" library="SparkFun" deviceset="GND" device=""/>
 <part name="Q1" library="murata-filter" deviceset="CSTCR" device="" technology="6M00G53Z"/>
-<part name="B1" library="SparkFun" deviceset="TAC_SWITCH" device="SMD" value="Button"/>
+<part name="BTN" library="SparkFun" deviceset="TAC_SWITCH" device="SMD" value="Button"/>
 <part name="GND27" library="SparkFun" deviceset="GND" device=""/>
+<part name="I2C" library="con-lstb" deviceset="MA04-1" device=""/>
+<part name="P+22" library="supply1" deviceset="VCC" device=""/>
+<part name="GND28" library="SparkFun" deviceset="GND" device=""/>
 </parts>
 <sheets>
@@
 <attribute name="VALUE" x="347.98" y="116.84" size="1.778" layer="96" rot="R180"/>
 </instance>
-<instance part="S2" gate="S" x="38.1" y="116.84" smashed="yes" rot="R90">
-<attribute name="NAME" x="32.766" y="120.142" size="1.778" layer="95"/>
+<instance part="RESET" gate="S" x="38.1" y="116.84" smashed="yes" rot="R90">
+<attribute name="NAME" x="25.146" y="115.062" size="1.778" layer="95"/>
 <attribute name="VALUE" x="42.672" y="113.284" size="1.778" layer="96" rot="R90"/>
 </instance>
@@
 <instance part="GND26" gate="1" x="129.54" y="91.44"/>
 <instance part="Q1" gate="G$1" x="50.8" y="78.74" rot="R270"/>
-<instance part="B1" gate="S" x="327.66" y="172.72" smashed="yes">
-<attribute name="NAME" x="330.962" y="178.054" size="1.778" layer="95" rot="R270"/>
-<attribute name="VALUE" x="324.104" y="168.148" size="1.778" layer="96"/>
+<instance part="BTN" gate="S" x="327.66" y="172.72" smashed="yes">
+<attribute name="NAME" x="327.406" y="178.562" size="1.778" layer="95"/>
+<attribute name="VALUE" x="324.104" y="165.608" size="1.778" layer="96"/>
 </instance>
 <instance part="GND27" gate="1" x="335.28" y="165.1"/>
+<instance part="I2C" gate="1" x="276.86" y="172.72" rot="R180"/>
+<instance part="P+22" gate="VCC" x="266.7" y="182.88" smashed="yes">
+<attribute name="VALUE" x="269.24" y="185.42" size="1.778" layer="96" rot="R180"/>
+</instance>
+<instance part="GND28" gate="1" x="266.7" y="165.1"/>
 </instances>
 <busses>
@@
 <wire x1="40.64" y1="109.22" x2="40.64" y2="106.68" width="0.1524" layer="91"/>
 <junction x="40.64" y="109.22"/>
-<pinref part="S2" gate="S" pin="1"/>
-<pinref part="S2" gate="S" pin="2"/>
+<pinref part="RESET" gate="S" pin="1"/>
+<pinref part="RESET" gate="S" pin="2"/>
 <pinref part="GND14" gate="1" pin="GND"/>
 </segment>
@@
 </segment>
 <segment>
-<pinref part="B1" gate="S" pin="4"/>
+<pinref part="BTN" gate="S" pin="4"/>
 <wire x1="332.74" y1="170.18" x2="335.28" y2="170.18" width="0.1524" layer="91"/>
 <wire x1="335.28" y1="170.18" x2="335.28" y2="172.72" width="0.1524" layer="91"/>
-<pinref part="B1" gate="S" pin="3"/>
+<pinref part="BTN" gate="S" pin="3"/>
 <wire x1="335.28" y1="172.72" x2="332.74" y2="172.72" width="0.1524" layer="91"/>
 <pinref part="GND27" gate="1" pin="GND"/>
 <wire x1="335.28" y1="170.18" x2="335.28" y2="167.64" width="0.1524" layer="91"/>
 <junction x="335.28" y="170.18"/>
+</segment>
+<segment>
+<pinref part="I2C" gate="1" pin="4"/>
+<wire x1="269.24" y1="170.18" x2="266.7" y2="170.18" width="0.1524" layer="91"/>
+<wire x1="266.7" y1="170.18" x2="266.7" y2="167.64" width="0.1524" layer="91"/>
+<pinref part="GND28" gate="1" pin="GND"/>
 </segment>
 </net>
@@
 <label x="123.19" y="26.67" size="1.778" layer="95" rot="R180"/>
 </segment>
+<segment>
+<pinref part="I2C" gate="1" pin="1"/>
+<wire x1="269.24" y1="177.8" x2="266.7" y2="177.8" width="0.1524" layer="91"/>
+<wire x1="266.7" y1="177.8" x2="266.7" y2="180.34" width="0.1524" layer="91"/>
+<pinref part="P+22" gate="VCC" pin="VCC"/>
+</segment>
 </net>
 <net name="VIBRATOR" class="0">
@@
 <label x="106.68" y="124.46" size="1.778" layer="95"/>
 </segment>
+<segment>
+<pinref part="I2C" gate="1" pin="2"/>
+<wire x1="269.24" y1="175.26" x2="264.16" y2="175.26" width="0.1524" layer="91"/>
+<junction x="264.16" y="175.26"/>
+<label x="254" y="175.26" size="2.1844" layer="95"/>
+</segment>
 </net>
 <net name="SCL" class="0">
@@
 <junction x="132.08" y="121.92"/>
 <label x="106.68" y="121.92" size="1.778" layer="95"/>
+</segment>
+<segment>
+<pinref part="I2C" gate="1" pin="3"/>
+<wire x1="269.24" y1="172.72" x2="264.16" y2="172.72" width="0.1524" layer="91"/>
+<junction x="264.16" y="172.72"/>
+<label x="254" y="172.72" size="2.1844" layer="95"/>
 </segment>
 </net>
@@
 <junction x="38.1" y="124.46"/>
 <pinref part="U5" gate="G$1" pin="PC6(/RESET)"/>
-<pinref part="S2" gate="S" pin="3"/>
-<pinref part="S2" gate="S" pin="4"/>
+<pinref part="RESET" gate="S" pin="3"/>
+<pinref part="RESET" gate="S" pin="4"/>
 <pinref part="R8" gate="G$1" pin="1"/>
 <pinref part="C11" gate="G$1" pin="2"/>
@@
 </segment>
 <segment>
-<pinref part="B1" gate="S" pin="2"/>
+<pinref part="BTN" gate="S" pin="2"/>
 <wire x1="322.58" y1="170.18" x2="320.04" y2="170.18" width="0.1524" layer="91"/>
 <wire x1="320.04" y1="170.18" x2="320.04" y2="172.72" width="0.1524" layer="91"/>
-<pinref part="B1" gate="S" pin="1"/>
+<pinref part="BTN" gate="S" pin="1"/>
 <wire x1="320.04" y1="172.72" x2="322.58" y2="172.72" width="0.1524" layer="91"/>
 <wire x1="320.04" y1="170.18" x2="317.5" y2="170.18" width="0.1524" layer="91"/>

Commit message: PCB Version 0.6.2
Parts:
- removed M1: ELECTRET_MICROPHON-F6035AP, microphon:ELECTRET_MICROPHON-F6035AP
- added MIC+, MIC-: (no value), wirepad:2,15/1,0
Connections:
- net N$2: now also MIC+.P; no longer M1.1
- net N$3: now also MIC-.P; no longer M1.2
Other:
- note added: "Charles Rincheval"
Changed lines of the file:
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@@
 <setting verticaltext="up"/>
 </settings>
-<grid distance="0.1" unitdist="inch" unit="inch" style="dots" multiple="1" display="yes" altdistance="0.01" altunitdist="inch" altunit="inch"/>
+<grid distance="0.1" unitdist="inch" unit="inch" style="lines" multiple="1" display="no" altdistance="0.01" altunitdist="inch" altunit="inch"/>
 <layers>
 <layer number="1" name="Top" color="4" fill="1" visible="no" active="no"/>
@@
 <part name="C6" library="rcl" deviceset="CPOL-EU" device="CT3528" value="10uf"/>
 <part name="C7" library="rcl" deviceset="CPOL-EU" device="CT3528" value="10uf"/>
-<part name="M1" library="microphon" deviceset="ELECTRET_MICROPHON-" device="F6035AP"/>
 <part name="C9" library="rcl" deviceset="C-EU" device="C0805" value="100nf"/>
 <part name="P+21" library="supply1" deviceset="VCC" device=""/>
@@
 <part name="P+22" library="supply1" deviceset="VCC" device=""/>
 <part name="GND28" library="SparkFun" deviceset="GND" device=""/>
+<part name="MIC+" library="wirepad" deviceset="2,15/1,0" device=""/>
+<part name="MIC-" library="wirepad" deviceset="2,15/1,0" device=""/>
 </parts>
 <sheets>
@@
 <text x="10.16" y="139.7" size="6.4516" layer="98">Core</text>
 <text x="248.92" y="243.84" size="6.4516" layer="98">Interface</text>
+<text x="347.98" y="20.32" size="2.54" layer="94">Charles Rincheval</text>
 </plain>
 <instances>
@@
 <instance part="C6" gate="G$1" x="269.24" y="134.62"/>
 <instance part="C7" gate="G$1" x="292.1" y="58.42"/>
-<instance part="M1" gate="G$1" x="355.6" y="73.66"/>
 <instance part="C9" gate="G$1" x="218.44" y="203.2" rot="R180"/>
 <instance part="P+21" gate="VCC" x="218.44" y="215.9" smashed="yes">
@@
 </instance>
 <instance part="GND28" gate="1" x="266.7" y="165.1"/>
+<instance part="MIC+" gate="1" x="353.06" y="73.66" smashed="yes" rot="R180">
+<attribute name="NAME" x="361.823" y="74.3458" size="1.778" layer="95" rot="R180"/>
+<attribute name="VALUE" x="354.203" y="76.962" size="1.778" layer="96" rot="R180"/>
+</instance>
+<instance part="MIC-" gate="1" x="353.06" y="71.12" smashed="yes" rot="R180">
+<attribute name="NAME" x="361.823" y="71.8058" size="1.778" layer="95" rot="R180"/>
+<attribute name="VALUE" x="354.203" y="74.422" size="1.778" layer="96" rot="R180"/>
+</instance>
 </instances>
 <busses>
@@
 <pinref part="R3" gate="G$1" pin="1"/>
 <pinref part="C19" gate="G$1" pin="2"/>
-<pinref part="M1" gate="G$1" pin="1"/>
+<pinref part="MIC+" gate="1" pin="P"/>
 </segment>
 </net>
@@
 <pinref part="R4" gate="G$1" pin="2"/>
 <pinref part="C20" gate="G$1" pin="1"/>
-<pinref part="M1" gate="G$1" pin="2"/>
-</segment>
-</net>
+<pinref part="MIC-" gate="1" pin="P"/>
+</segment>
+</net>
