File: pcb/mds.sch (EAGLE design)
At the start: 51 parts, among them IC1 MAX1555, Q1 CSTCR6M00G53Z, U2 ISD1900ISD1932, U5 ATMEGA328

Commit message: Code + Doc + OpenScad
Parts:
- removed T1: (no value), transistor:-NPN-SOT23-EBC
- added T2: (no value), transistor-neu-to92:MMBT2222ALT1-NPN-SOT23-BEC
- R1, R5, R7: value (none) -> 4.7k
Connections:
- net GND: now also T2.E; no longer T1.E
- net N$5: now also T2.B; no longer T1.B
- net N$7: now also T2.C; no longer T1.C
Changed lines of the file:
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@@
 <part name="U$13" library="gy-27" deviceset="GY-27" device=""/>
 <part name="U$14" library="SparkFun" deviceset="OSHW-LOGO" device="S"/>
-<part name="T1" library="transistor" deviceset="*-NPN-" device="SOT23-EBC"/>
 <part name="GND10" library="SparkFun" deviceset="GND" device=""/>
 <part name="GND12" library="SparkFun" deviceset="GND" device=""/>
-<part name="R5" library="rcl" deviceset="R-EU_" device="M0805"/>
+<part name="R5" library="rcl" deviceset="R-EU_" device="M0805" value="4.7k"/>
 <part name="MOT-" library="wirepad" deviceset="2,15/1,0" device=""/>
 <part name="MOT+" library="wirepad" deviceset="2,15/1,0" device=""/>
@@
 <part name="P+14" library="supply1" deviceset="VCC" device=""/>
 <part name="P+19" library="supply1" deviceset="VCC" device=""/>
-<part name="R1" library="rcl" deviceset="R-EU_" device="M0805"/>
-<part name="R7" library="rcl" deviceset="R-EU_" device="M0805"/>
+<part name="R1" library="rcl" deviceset="R-EU_" device="M0805" value="4.7k"/>
+<part name="R7" library="rcl" deviceset="R-EU_" device="M0805" value="4.7k"/>
 <part name="P+20" library="supply1" deviceset="VCC" device=""/>
 <part name="P+13" library="supply1" deviceset="VCC" device=""/>
@@
 <part name="MIC+" library="wirepad" deviceset="2,15/1,0" device=""/>
 <part name="MIC-" library="wirepad" deviceset="2,15/1,0" device=""/>
+<part name="T2" library="transistor-neu-to92" deviceset="*-NPN-" device="SOT23-BEC" technology="MMBT2222ALT1"/>
 </parts>
 <sheets>
@@
 <instance part="U$13" gate="G$1" x="195.58" y="198.12"/>
 <instance part="U$14" gate="G$1" x="271.78" y="15.24"/>
-<instance part="T1" gate="G$1" x="292.1" y="203.2"/>
 <instance part="GND10" gate="1" x="294.64" y="193.04"/>
 <instance part="GND12" gate="1" x="210.82" y="190.5"/>
@@
 <attribute name="VALUE" x="354.203" y="74.422" size="1.778" layer="96" rot="R180"/>
 </instance>
+<instance part="T2" gate="G$1" x="292.1" y="203.2"/>
 </instances>
 <busses>
@@
 </segment>
 <segment>
-<pinref part="T1" gate="G$1" pin="E"/>
 <pinref part="GND10" gate="1" pin="GND"/>
 <wire x1="294.64" y1="195.58" x2="294.64" y2="198.12" width="0.1524" layer="91"/>
+<pinref part="T2" gate="G$1" pin="E"/>
 </segment>
 <segment>
@@
 <net name="N$5" class="0">
 <segment>
-<pinref part="T1" gate="G$1" pin="B"/>
 <pinref part="R5" gate="G$1" pin="2"/>
 <wire x1="287.02" y1="203.2" x2="289.56" y2="203.2" width="0.1524" layer="91"/>
+<pinref part="T2" gate="G$1" pin="B"/>
 </segment>
 </net>
 <net name="N$7" class="0">
 <segment>
-<pinref part="T1" gate="G$1" pin="C"/>
 <wire x1="294.64" y1="208.28" x2="294.64" y2="210.82" width="0.1524" layer="91"/>
 <pinref part="MOT-" gate="1" pin="P"/>
 <wire x1="294.64" y1="210.82" x2="297.18" y2="210.82" width="0.1524" layer="91"/>
-</segment>
-</net>
+<pinref part="T2" gate="G$1" pin="C"/>
+</segment>
+</net>
