File: pcb/mds.sch (EAGLE design)
At the start: 62 parts, among them IC1 MAX1555, Q2 MOSFET-P, U2 ISD1900ISD1932, U3 ADXL345, U5 ATMEGA328

Commit message: Update CAD
Parts:
- removed D4: (no value), OPL Eagle Library:D-D1206
- added D1: 1N4148, OPL Eagle Library:D-D1206
- added R16: 33k, rcl:R-EU_M0805
- added R17: 2.2k, rcl:R-EU_M0805
- added T1: (no value), transistor-neu-to92:MMBT2222ALT1-NPN-SOT23-BEC
- D3: value (none) -> Schottky
- R10: value 4.7k -> 1.2M
Connections:
- new net N$4: R16.1, T1.B
- new net PWR_STATUS: D1.+, U5.PD3(INT1)
- net CHG: now also D1.-; no longer U5.PD3(INT1)
- net GND: now also R17.2, T1.E
- net N$9: now also Q2.G, R10.1, T1.C; no longer D4.-
- net PWR_CMD: now also R16.2, R17.1; no longer D3.+, D4.+, Q2.G, R10.1
Other:
- note added: "If CHG goes DOWN, then power up ! If PWR_CMD goes UP, then power up !"
- note removed: "If CHG, then power up !"
- moved on the sheet: C18, Q2, R10
