File: pcb/mds2.brd (EAGLE design)
At the start: 73 x 41.9 mm, 126 parts, among them CN1 2908-05WB-M6, IC2 MAX1555, Q2 MOSFET-P, U1 ATMEGA32U4, U10 LSM303DLHC, U11 BMP180, U6 VS1053B, U7 AP7312-1833W6-7, U9 L3GD20, Y1 8MHz, Y2 ABM8G-12.288MHZ-4Y-T3

Commit message: Work on Schematic / PCB
Parts:
- removed CN1: 2908-05WB-M6, microbuilder:MICROSD
- removed D1: Green, SparkFun:LED-0603
- removed PAD1, PAD2, PAD3, PAD4, PAD5, PAD6: WIREPADSMD1,27-254, wirepad:SMD1,27-2,54
- removed P_3V3, P_GND, P_MISO, P_MOSI, P_RESET, P_SCK: TPTP13R, testpad:TP13R
- removed SV1: (no value), con-lstb:MA03-2
- added C39: 100nf, rcl:C0805
- added ISP: (no value), con-lsta:FE06
- added J_AIN: (no value), jumper:SJ_2
- added LINE+, LINE-: (no value), wirepad:1,6/0,8
- added R33: 10k, rcl:M0805
- added STEPUP+, STEPUP-: (no value), wirepad:2,15/1,0
- added µSD: 2908-05WB-M6, microbuilder:MICROSD
- C22, C27: value 0.1µF -> 100nf; device microbuilder:_0805MP -> rcl:C0805
- FB1, FB2: value FERITTE -> FERITTE - 180Ω@100MHz
- R6: value 330 -> 10k
- moved RGB 42.0 mm to (44.6, 39.4), turned to 0 degrees
- moved R6 37.8 mm to (41.1, 26.8), turned to 90 degrees
- moved R9 19.7 mm to (47.6, 34.6), turned to 90 degrees
- moved R5 14.3 mm to (15.2, 35.6), turned to 90 degrees
- moved R12 10.2 mm to (58.6, 38.9)
- moved R18 9.26 mm to (54.6, 5.24), turned to 90 degrees
- moved R17 8.31 mm to (53.7, 14.4), turned to 270 degrees
- moved C2 8.11 mm to (22.5, 20.2), turned to 180 degrees
- moved R16 6.57 mm to (33.2, 10.2), turned to 90 degrees
- moved R20 6.19 mm to (55.6, 8.26), turned to 180 degrees
- moved FB1 6.13 mm to (33.5, 21.4), turned to 270 degrees
- moved R11 5.94 mm to (60.6, 38.9), turned to 270 degrees
- moved C5 5.78 mm to (53.7, 30.6), turned to 180 degrees
- moved R19 5.40 mm to (55.6, 14.4), turned to 270 degrees
- moved C23 5.02 mm to (43.5, 27.0)
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Connections:
- removed net D13_LED_RED: R6.1
- removed net LINE2: U6.48
- removed net N$15: PAD4.1, PAD5.1, PAD6.1
- removed net N$6: D1.A, R6.2
- removed net SCK: P_SCK.TP
- removed net TXLED: U1.22
- removed net _CHG: U1.33
- new net LINE+: J_AIN.3, LINE+.1
- new net LINE-: LINE-.1, U6.48
- new net N$16: J_AIN.2, U6.1
- new net SHUTDOWN: AMPLIFIER.2, R33.2, U1.33
- net +3V3: now also ISP.3, R16.2, R6.1, µSD.4; no longer AMPLIFIER.2, CN1.4, P_3V3.TP
- net AGND: now also C22.1, R33.1; no longer C22.2
- net AVDD: now also C22.2; no longer C22.1, R16.2
- net GND: now also C27.1, C39.1, ISP.2, µSD.6, µSD.MT1, µSD.MT2; no longer C27.2, CN1.6, CN1.MT1, CN1.MT2, D1.C, P_GND.TP
- net LEFT: now also R17.2, R19.2; no longer R18.2, R20.2
- net LEFT_FILTERED: now also R19.1; no longer R20.1
- net MIC+: now also J_AIN.1; no longer U6.1
- net MISO: now also ISP.5, µSD.7; no longer CN1.7, P_MISO.TP
- net MOSI: now also ISP.6, µSD.3; no longer CN1.3, P_MOSI.TP
- net N$31: now also R17.1; no longer R18.1
- net N$32: now also R18.1; no longer R17.1
- net RESET: now also ISP.4; no longer P_RESET.TP
- net RIGHT: now also R18.2, R20.2; no longer R17.2, R19.2
- net RIGHT_FILTERED: now also R20.1; no longer R19.1
- net RST: now also C27.2; no longer C27.1
- net SCLK: now also ISP.1, µSD.5; no longer CN1.5
- net SD_DETECT: now also R6.2, U1.39, µSD.CD1; no longer CN1.CD1
- net VCC: now also C39.2, STEPUP+.1, STEPUP-.1
- net _SDCS_NC: now also µSD.2; no longer CN1.2
Routing:
- net +3V3: track 58.7 -> 188.9 mm, vias 4 -> 18
- net VCC: track 5.90 -> 105.5 mm, vias 0 -> 7
- net SHUTDOWN: track 0.00 -> 82.2 mm, vias 0 -> 3
- net MISO: track 41.3 -> 101.3 mm, vias 1 -> 5
- net PWR_CMD: track 2.54 -> 58.9 mm, vias 0 -> 4
- net CHG: track 11.1 -> 64.7 mm, vias 2 -> 4
- net V_PWR: track 3.34 -> 51.5 mm, vias 0 -> 4
- net SCLK: track 24.5 -> 71.8 mm, vias 1 -> 5
- net LED_STRIP: track 0.00 -> 46.6 mm, vias 0 -> 5
- net MOSI: track 38.2 -> 81.5 mm, vias 1 -> 5
- net N$3: track 22.6 -> 65.0 mm, vias 0 -> 3
- net D5_LED_GREEN: track 0.00 -> 40.2 mm, vias 0 -> 4
- net AVDD: track 6.69 -> 42.2 mm, vias 2 -> 4
- net CS: track 18.3 -> 52.2 mm, vias 2 -> 4
- net RST: track 18.3 -> 50.5 mm, vias 1 -> 3
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Other:
- outline, holes or cut-outs redrawn
- board text added: "+3V3"
- board text added: "MISO"
- board text added: "MOSI"
- board text added: "RESET"
- board text added: "SCLK"
- board text added: "Todo: Faire des ponts par défaut sur les jumper CMS"

Commit message: Add PCB 2.0.0
Parts:
- removed I2C: (no value), con-lstb:MA04-1
- removed ISP: (no value), con-lsta:FE06
- removed J_CHG: (no value), jumper:SJ_2
- removed RGB: (no value), con-lstb:MA03-1
- added ADC0, ADC1: TPB1,27, testpad:B1,27
- added BAT+, BAT-, WUP: (no value), wirepad:1,6/0,8
- added C40, C41: 10uf, rcl:C0805
- added C42: 100nf, rcl:C0805
- added C43, C44: 10pf, rcl:C0805
- added D1: BAT54C, diode:SOT23
- added EXT: (no value), con-lstb:MA05-1
- added FB3: FERITTE - 180Ω@100MHz, microbuilder:_0805MP
- added IO1: MCP79410_MSOP8, timers-clocks:MSOP8
- added ISP6: (no value), con-lstb:MA03-2
- added J_PRG: (no value), jumper:SJ
- added Q6: 32.768khz, crystal:TC26H
- added STRIP: (no value), con-lstb:MA03-1
- C26, C37: device rcl:PANASONIC_B -> rcl:PANASONIC_C
- C28, C29: value 220uF -> 220uf; device rcl:PANASONIC_C -> rcl:PANASONIC_D
- C35: value 4.7uF -> 4.7uF (low ESR)
- C36: value 0.22µF -> 0.22µF (low ESR)
- D2: value Schottky -> BAT54A; device OPL Eagle Library:LL-34 -> diode:SOT23
- T1, T2: value (none) -> MMBT2222A
- moved U11 6.48 mm to (11.3, 3.33)
- moved R24 5.25 mm to (17.0, 5.56), turned to 0 degrees
- moved R22 5.08 mm to (64.0, 22.7)
- moved T2 5.08 mm to (17.0, 2.38), turned to 180 degrees
- moved VIB+ 4.33 mm to (20.5, 4.13)
- moved VIB- 4.33 mm to (20.5, 1.59)
- moved C33 2.72 mm to (12.9, 7.78), turned to 90 degrees
- moved C11 2.13 mm to (65.2, 17.9)
- moved C10 2.13 mm to (65.2, 20.0)
- moved R4 2.06 mm to (64.5, 26.2), turned to 180 degrees
- moved R28 1.59 mm to (61.6, 27.0)
- moved C22 0.96 mm to (33.6, 17.0)
- moved R5 0.95 mm to (15.2, 36.5)
- moved R9 0.95 mm to (48.6, 34.6)
- moved C12 0.85 mm to (62.4, 18.5)
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- renumbered µSD to MICROSD
Connections:
- net D5_LED_GREEN renamed LED
- removed net _SDCS_NC: MICROSD.2
- new net N$15: ADC1.TP, U1.40
- new net N$21: ADC0.TP, U1.41
- new net N$22: C44.1, IO1.2, Q6.1
- new net N$27: C43.1, IO1.1, Q6.2
- new net N$37: BAT+.1, IO1.3
- new net N$6: C39.2, C40.2, FB3.1, STRIP.1
- new net SDCS: MICROSD.2, U1.22
- new net TIMER: D2.1, IO1.7
- net +3V3: now also C42.2, EXT.2, IO1.8, J_PRG.2; no longer I2C.2, ISP.3
- net CHG: now also D2.2; no longer D2.C
- net GND: now also BAT-.1, C40.1, C41.1, C42.1, C43.2, C44.2, EXT.1, IO1.4, ISP6.6, STRIP.3, USB.BODY@1, USB.BODY@2, USB.BODY@3, USB.BODY@4; no longer I2C.1, ISP.2, RGB.3
- net LED_STRIP: now also STRIP.2; no longer RGB.2
- net MISO: now also ISP6.1; no longer ISP.5
- net MOSI: now also ISP6.4; no longer ISP.6
- net N$10: now also D2.3; no longer D2.A
- net N$11: now also D1.3, R28.1, R4.2; no longer C17.2, IC2.1, J_CHG.3
- net N$12: now also D1.2, WUP.1; no longer C16.2, IC2.4, J_CHG.1
- net N$3: now also C16.2, IC2.4; no longer J_CHG.2
- net PWR_CMD: now also D1.1; no longer R28.1, R4.2
- net RESET: now also ISP6.5; no longer ISP.4
- net SCL: now also EXT.5, IO1.6; no longer I2C.4
- net SCLK: now also ISP6.3; no longer ISP.1
- net SDA: now also EXT.4, IO1.5; no longer I2C.3
- net VBUS: now also C17.2, IC2.1
- net VCC: now also C41.2, EXT.3, FB3.2, ISP6.2, J_PRG.1; no longer C39.2, RGB.1
Routing:
- net TIMER: track 0.00 -> 73.3 mm, vias 0 -> 4
- net VBUS: track 16.9 -> 80.1 mm, vias 0 -> 5
- net SDCS: track 0.00 -> 32.2 mm, vias 0 -> 2
- net VCC: track 105.5 -> 133.7 mm, vias 7 -> 10
- net SCLK: track 71.8 -> 89.9 mm, vias 5 -> 6
- net MOSI: track 81.5 -> 95.4 mm
- net N$37: track 0.00 -> 13.0 mm, vias 0 -> 1
- net +3V3: track 188.9 -> 199.5 mm, vias 18 -> 17
- net CS: track 52.2 -> 62.8 mm
- net N$22: track 0.00 -> 8.65 mm
- net GND: track 58.1 -> 65.7 mm, vias 38 -> 76
- net N$6: track 0.00 -> 7.09 mm
- net N$12: track 8.47 -> 2.05 mm, vias 1 -> 0
- net SCL: track 44.4 -> 50.3 mm
- net N$27: track 0.00 -> 5.40 mm
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Other:
- outline, holes or cut-outs redrawn
- board text added: "(max 7V)"
- board text added: "+"
- board text added: "-"
- board text added: "15dB"
- board text added: "3V3"
- board text added: "9dB"
- board text added: "Audio out"
- board text added: "CHARGER"
- board text added: "Charge"
- board text added: "DRDY"
- board text added: "For use : 1. Cut the bridge 2. Connect reg"
- board text added: "GND"
- board text added: "IN"
- board text added: "INT1"
- board text added: "INT2"
- board text added: "ISP"
- board text added: "LEFT"
- board text added: "LINE"
- board text added: "LIPO"
- board text added: "Led strip"
- board text added: "LiPo"
- board text added: "MIC"
- board text added: "MurmureDuSon"
- board text added: "OUT"
- board text added: "RDY"
- board text added: "RIGHT"
- board text added: "RTC Backup"
- board text added: "SCL"
- board text added: "SDA"
- board text added: "StepUp In"
- board text added: "VCC"
- board text added: "Vibrating motor"
- board text added: "WUP"
- board text added: "WakeUp"
- board text added: "hugo, 05/2016 www.digitalspirit.org"
- board text added: "v2.0.x"
- board text removed: "+3V3"
- board text removed: "MISO"
- board text removed: "MOSI"
- board text removed: "RESET"
- board text removed: "SCLK"
- board text removed: "Todo: Faire des ponts par défaut sur les jumper CMS"
- board text removed: "Todo: Faire des trous pour la fixation de la LiPo"
- board text removed: "Todo: Vérifier le connecteur ISP"
- board text removed: "Todo: Vérifier le diamètre / position des trous de montage"
- board text removed: "Todo: Vérifier les trous pour le vibreur"
