File: pcb/mds2.sch (EAGLE design)
At the start: 126 parts, among them CN1 2908-05WB-M6, IC2 MAX1555, Q2 MOSFET-P, U1 ATMEGA32U4, U10 LSM303DLHC, U11 BMP180, U6 VS1053B, U7 AP7312-1833W6-7, U9 L3GD20, Y1 8MHz, Y2 ABM8G-12.288MHZ-4Y-T3

Commit message: Work on Schematic / PCB
Parts:
- removed D1: Green, SparkFun:LED0603
- removed PAD1, PAD2, PAD3, PAD4, PAD5, PAD6: WIREPADSMD1,27-254, wirepad:WIREPADSMD1,27-254
- removed P_3V3, P_GND, P_MISO, P_MOSI, P_RESET, P_SCK: TPTP13R, testpad:TPTP13R
- removed SV1: (no value), con-lstb:MA03-2
- added C39: 100nf, rcl:C-EUC0805
- added ISP: (no value), con-lsta:FE06-1
- added J_AIN: (no value), jumper:SJ2W
- added LINE+, LINE-: (no value), wirepad:1,6/0,8
- added R33: 10k, rcl:R-EU_M0805
- added STEPUP+, STEPUP-: (no value), wirepad:2,15/1,0
- C22, C27: value 0.1µF -> 100nf; device microbuilder:CAP_CERAMIC_0805MP -> rcl:C-EUC0805
- FB1, FB2: value FERITTE -> FERITTE - 180Ω@100MHz
- R6: value 330 -> 10k
- renumbered CN1 to µSD
Connections:
- removed net D13_LED_RED: R6.1
- removed net LINE2: U6.LINE2
- removed net N$15: PAD4.P, PAD5.P, PAD6.P
- removed net N$6: D1.A, R6.2
- removed net SCK: P_SCK.TP
- removed net TXLED: U1.PD5
- removed net _CHG: U1.PE2/!HWB
- new net LINE+: J_AIN.3, LINE+.P
- new net LINE-: LINE-.P, U6.LINE2
- new net N$16: J_AIN.2, U6.MIC_P/LINEIN
- new net SHUTDOWN: AMPLIFIER.SHDN, R33.2, U1.PE2/!HWB
- net +3V3: now also ISP.3, R16.2, R6.1; no longer AMPLIFIER.SHDN, P_3V3.TP
- net AGND: now also C22.1, R33.1; no longer C22.2
- net AVDD: now also C22.2; no longer C22.1, R16.2
- net GND: now also C27.1, C39.1, ISP.2; no longer C27.2, D1.C, P_GND.TP
- net LEFT: now also R17.2, R19.2; no longer R18.2, R20.2
- net LEFT_FILTERED: now also R19.1; no longer R20.1
- net MIC+: now also J_AIN.1; no longer U6.MIC_P/LINEIN
- net MISO: now also ISP.5; no longer P_MISO.TP
- net MOSI: now also ISP.6; no longer P_MOSI.TP
- net N$31: now also R17.1; no longer R18.1
- net N$32: now also R18.1; no longer R17.1
- net RESET: now also ISP.4; no longer P_RESET.TP
- net RIGHT: now also R18.2, R20.2; no longer R17.2, R19.2
- net RIGHT_FILTERED: now also R20.1; no longer R19.1
- net RST: now also C27.2; no longer C27.1
- net SCLK: now also ISP.1
- net SD_DETECT: now also R6.2, U1.PF4(ADC4)
- net VCC: now also C39.2, STEPUP+.P, STEPUP-.P
Other:
- note added: "Optional Step-Up connector Cut the bridge / connect power"
- note removed: "TODO: Ajouter le circuit du MIC"
- note removed: "TODO: Mettre un module I2C RTC ?"
- note removed: "TODO: Prévoir un moyen avec un pont pur injecter une DC/DC StepUp"
- note removed: "TODO: Si il reste une IO libre sur l'avr, l'utiliser pour le shutdown"
- moved on the sheet: C20, C21, C22, C27, LIPO+, LIPO-, R16, R18, R19, R20, R24, R25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

Commit message: Add PCB 2.0.0
Parts:
- removed I2C: (no value), con-lstb:MA04-1
- removed ISP: (no value), con-lsta:FE06-1
- removed J_CHG: (no value), jumper:SJ2W
- removed RGB: (no value), con-lstb:MA03-1
- added ADC0, ADC1: TPB1,27, testpad:TPB1,27
- added BAT+, BAT-, WUP: (no value), wirepad:1,6/0,8
- added C40, C41: 10uf, rcl:C-EUC0805
- added C42: 100nf, rcl:C-EUC0805
- added C43, C44: 10pf, rcl:C-EUC0805
- added D1: BAT54C, diode:BAT54C
- added EXT: (no value), con-lstb:MA05-1
- added FB3: FERITTE - 180Ω@100MHz, microbuilder:FERRITE_0805MP
- added IO1: MCP79410_MSOP8, timers-clocks:MCP79410_MSOP8
- added ISP6: (no value), con-lstb:MA03-2
- added J_PRG: (no value), jumper:SJ
- added Q6: 32.768khz, crystal:CRYSTALTC26H
- added STRIP: (no value), con-lstb:MA03-1
- C26, C37: device rcl:CPOL-EUB -> rcl:CPOL-EUC
- C28, C29: value 220uF -> 220uf; device rcl:CPOL-USC -> rcl:CPOL-EUD
- C35: value 4.7uF -> 4.7uF (low ESR)
- C36: value 0.22µF -> 0.22µF (low ESR)
- D2: value Schottky -> BAT54A; device OPL Eagle Library:D-D1206 -> diode:BAT54A
- T1, T2: value (none) -> MMBT2222A
- renumbered µSD to MICROSD
Connections:
- net D5_LED_GREEN renamed LED
- removed net _SDCS_NC: MICROSD.CS
- new net N$15: ADC1.TP, U1.PF1(ADC1)
- new net N$21: ADC0.TP, U1.PF0(ADC0)
- new net N$22: C44.1, IO1.X2, Q6.1
- new net N$27: C43.1, IO1.X1, Q6.2
- new net N$37: BAT+.P, IO1.VBAT
- new net N$6: C39.2, C40.2, FB3.P$1, STRIP.1
- new net SDCS: MICROSD.CS, U1.PD5
- new net TIMER: D2.K1, IO1.MFP
- net +3V3: now also C42.2, EXT.2, IO1.VCC, J_PRG.2; no longer I2C.2, ISP.3
- net CHG: now also D2.K2; no longer D2.-
- net GND: now also BAT-.P, C40.1, C41.1, C42.1, C43.2, C44.2, EXT.1, IO1.VSS, ISP6.6, STRIP.3, USBBODY.BODY@1, USBBODY.BODY@2, USBBODY.BODY@3, USBBODY.BODY@4; no longer I2C.1, ISP.2, RGB.3
- net LED_STRIP: now also STRIP.2; no longer RGB.2
- net MISO: now also ISP6.1; no longer ISP.5
- net MOSI: now also ISP6.4; no longer ISP.6
- net N$10: now also D2.AA; no longer D2.+
- net N$11: now also D1.CC, R28.1, R4.2; no longer C17.2, IC2.USB, J_CHG.3
- net N$12: now also D1.A2, WUP.P; no longer C16.2, IC2.DC, J_CHG.1
- net N$3: now also C16.2, IC2.DC; no longer J_CHG.2
- net PWR_CMD: now also D1.A1; no longer R28.1, R4.2
- net RESET: now also ISP6.5; no longer ISP.4
- net SCL: now also EXT.5, IO1.SCL; no longer I2C.4
- net SCLK: now also ISP6.3; no longer ISP.1
- net SDA: now also EXT.4, IO1.SDA; no longer I2C.3
- net VBUS: now also C17.2, IC2.USB
- net VCC: now also C41.2, EXT.3, FB3.P$2, ISP6.2, J_PRG.1; no longer C39.2, RGB.1
Other:
- note added: "If CHG / TIMER goes DOWN, then power up ! If PWR_CMD or WUP (WakeUp) goes UP, then power up !"
- note added: "Program AVR without any other chip"
- note added: "RTC"
- note added: "TODO: Vérifier les adresses du bus I2C"
- note removed: "Alim en 3V ou plus ?"
- note removed: "If CHG goes DOWN, then power up ! If PWR_CMD goes UP, then power up !"
- note removed: "TODO: Mettre des filtres (capa / feritte) proche de l'alim du led strip"
- note removed: "TODO: Vérifier que les condos B sont bon en 10uf"
- moved on the sheet: C16, C17, C39, CHG+, CHG-, D3, R10, R13, R14, R24, R5, T2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
